File: hardware/pcb/audiostick_v1.sch (EAGLE design)
At the start: 56 parts, among them IC3 PCM5102ASW, IC5 AP22804W5, IC6 TINY13V-10SSU, J1 AVRISP6TH127, J2 AUDIO_JACK_3.5MM_PTH, J3 USB-B

Commit message: first v2 commit
Parts:
- C16, C4: value 10n -> 100n
