File: hardware/pcb/audiostick.kicad_pcb (KiCad board)
At the start: 2 copper layers, 74 x 33.5 mm, 61 parts, among them J1 USB_B_Micro, J2 Conn_02x20_Odd_Even, J3 AudioJack3_Switch, SW1 SW_Push, U1 AP2127K-3.3, U2 AP2161W, U3 PCM5102, U4 ATtiny202-SS, U5 AT24CS01-STUM

Commit message: Removed external EEPROM, some layout changes
Parts:
- moved FID2 0.50 mm to (178.0, 92.0)
Routing:
- net +3.3VA: track 81.2 -> 82.1 mm
- net GND: vias 45 -> 54
Changed lines of the file:
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@@
   (general
     (thickness 1.6)
-    (drawings 11)
-    (tracks 282)
+    (drawings 13)
+    (tracks 291)
     (zones 0)
     (modules 61)
@@
   )
   (setup
-    (last_trace_width 0.3)
+    (last_trace_width 0.25)
     (user_trace_width 0.3)
     (user_trace_width 0.5)
@@
     (add_net "Net-(C3-Pad1)")
     (add_net "Net-(D1-Pad2)")
-    (add_net "Net-(J1-Pad2)")
-    (add_net "Net-(J1-Pad3)")
-    (add_net "Net-(J1-Pad4)")
-    (add_net "Net-(J2-Pad10)")
-    (add_net "Net-(J2-Pad12)")
-    (add_net "Net-(J2-Pad13)")
-    (add_net "Net-(J2-Pad14)")
-    (add_net "Net-(J2-Pad15)")
-    (add_net "Net-(J2-Pad17)")
-    (add_net "Net-(J2-Pad18)")
-    (add_net "Net-(J2-Pad19)")
-    (add_net "Net-(J2-Pad20)")
-    (add_net "Net-(J2-Pad22)")
-    (add_net "Net-(J2-Pad23)")
-    (add_net "Net-(J2-Pad24)")
-    (add_net "Net-(J2-Pad25)")
-    (add_net "Net-(J2-Pad26)")
-    (add_net "Net-(J2-Pad27)")
-    (add_net "Net-(J2-Pad3)")
-    (add_net "Net-(J2-Pad31)")
-    (add_net "Net-(J2-Pad33)")
-    (add_net "Net-(J2-Pad34)")
-    (add_net "Net-(J2-Pad36)")
-    (add_net "Net-(J2-Pad38)")
-    (add_net "Net-(J2-Pad4)")
-    (add_net "Net-(J2-Pad40)")
-    (add_net "Net-(J2-Pad5)")
-    (add_net "Net-(J2-Pad8)")
-    (add_net "Net-(J2-Pad9)")
-    (add_net "Net-(J3-PadTN)")
     (add_net "Net-(R7-Pad1)")
     (add_net "Net-(R8-Pad1)")
@@
     (add_net "Net-(TP13-Pad1)")
     (add_net "Net-(TP16-Pad1)")
-    (add_net "Net-(U1-Pad4)")
-    (add_net "Net-(U2-Pad3)")
     (add_net VBUS)
   )
@@
   )
   (module Fiducial:Fiducial_1mm_Mask2mm (layer F.Cu)
-    (at 178 91.5)
+    (at 178 92)
     (descr "Circular Fiducial, 1mm bare copper, 2mm soldermask opening (Level A)")
     (tags fiducial)
@@
       (rotate (xyz 0 0 0))
     )
+  )
+  (dimension 34 (width 0.15) (layer Dwgs.User)
+    (gr_text "34.000 mm" (at 221.3 78 90) (layer Dwgs.User)
+      (effects (font (size 1 1) (thickness 0.15)))
+    )
+    (feature1 (pts (xy 210 61) (xy 220.586421 61)))
+    (feature2 (pts (xy 210 95) (xy 220.586421 95)))
+    (crossbar (pts (xy 220 95) (xy 220 61)))
+    (arrow1a (pts (xy 220 61) (xy 220.586421 62.126504)))
+    (arrow1b (pts (xy 220 61) (xy 219.413579 62.126504)))
+    (arrow2a (pts (xy 220 95) (xy 220.586421 93.873496)))
+    (arrow2b (pts (xy 220 95) (xy 219.413579 93.873496)))
+  )
+  (dimension 74 (width 0.15) (layer Dwgs.User)
+    (gr_text "74.000 mm" (at 167 111.3) (layer Dwgs.User)
+      (effects (font (size 1 1) (thickness 0.15)))
+    )
+    (feature1 (pts (xy 204 100) (xy 204 110.586421)))
+    (feature2 (pts (xy 130 100) (xy 130 110.586421)))
+    (crossbar (pts (xy 130 110) (xy 204 110)))
+    (arrow1a (pts (xy 204 110) (xy 202.873496 110.586421)))
+    (arrow1b (pts (xy 204 110) (xy 202.873496 109.413579)))
+    (arrow2a (pts (xy 130 110) (xy 131.126504 110.586421)))
+    (arrow2b (pts (xy 130 110) (xy 131.126504 109.413579)))
   )
   (gr_text BOTTOM (at 198 94) (layer B.Cu)
@@
   (via (at 158 94) (size 0.6) (drill 0.3) (layers F.Cu B.Cu) (net 1))
   (via (at 146 91) (size 0.6) (drill 0.3) (layers F.Cu B.Cu) (net 1))
-  (via (at 150 91) (size 0.6) (drill 0.3) (layers F.Cu B.Cu) (net 1))
+  (via (at 150.5 91) (size 0.6) (drill 0.3) (layers F.Cu B.Cu) (net 1))
   (via (at 148 82) (size 0.6) (drill 0.3) (layers F.Cu B.Cu) (net 1))
   (via (at 141 76.5) (size 0.6) (drill 0.3) (layers F.Cu B.Cu) (net 1))
@@
   (via (at 174 74) (size 0.6) (drill 0.3) (layers F.Cu B.Cu) (net 1))
   (via (at 175.5 83) (size 0.6) (drill 0.3) (layers F.Cu B.Cu) (net 1))
+  (via (at 148 84) (size 0.6) (drill 0.3) (layers F.Cu B.Cu) (net 1))
+  (via (at 146 82) (size 0.6) (drill 0.3) (layers F.Cu B.Cu) (net 1))
+  (via (at 150 82) (size 0.6) (drill 0.3) (layers F.Cu B.Cu) (net 1))
+  (via (at 148 86) (size 0.6) (drill 0.3) (layers F.Cu B.Cu) (net 1))
+  (via (at 146 90) (size 0.6) (drill 0.3) (layers F.Cu B.Cu) (net 1))
+  (via (at 150.5 90) (size 0.6) (drill 0.3) (layers F.Cu B.Cu) (net 1))
+  (via (at 147.5 92) (size 0.6) (drill 0.3) (layers F.Cu B.Cu) (net 1))
+  (via (at 149 92) (size 0.6) (drill 0.3) (layers F.Cu B.Cu) (net 1))
+  (via (at 154 85.25) (size 0.6) (drill 0.3) (layers F.Cu B.Cu) (net 1))
+  (via (at 181.5 88) (size 0.8) (drill 0.4) (layers F.Cu B.Cu) (net 2))
+  (segment (start 181.5 88) (end 183 88) (width 0.25) (layer B.Cu) (net 2))
   (via (at 162.25 84.25) (size 0.8) (drill 0.4) (layers F.Cu B.Cu) (net 3))
   (via (at 162.25 86.25) (size 0.8) (drill 0.4) (layers F.Cu B.Cu) (net 3))
-  (via (at 181.5 88) (size 0.8) (drill 0.4) (layers F.Cu B.Cu) (net 2))
-  (segment (start 181.5 88) (end 183 88) (width 0.25) (layer B.Cu) (net 2))
   (segment (start 158.7125 84.5) (end 158.75 84.5375) (width 0.3) (layer F.Cu) (net 3))
   (segment (start 157 84.5) (end 158.7125 84.5) (width 0.3) (layer F.Cu) (net 3))
@@
   (segment (start 155.25 92) (end 155.25 89.1) (width 0.5) (layer F.Cu) (net 9))
   (via (at 155.25 92) (size 0.8) (drill 0.4) (layers F.Cu B.Cu) (net 9))
-  (segment (start 154.850001 92.399999) (end 141.149999 92.399999) (width 0.5) (layer B.Cu) (net 9))
-  (segment (start 155.25 92) (end 154.850001 92.399999) (width 0.5) (layer B.Cu) (net 9))
-  (segment (start 140.5 91.75) (end 140.5 89.5) (width 0.5) (layer B.Cu) (net 9))
-  (segment (start 141.149999 92.399999) (end 140.5 91.75) (width 0.5) (layer B.Cu) (net 9))
   (segment (start 140.6 89.4) (end 140.5 89.5) (width 0.5) (layer F.Cu) (net 9))
   (segment (start 141.75 89.4) (end 140.6 89.4) (width 0.5) (layer F.Cu) (net 9))
@@
   (segment (start 189.3 81.45) (end 189.25 81.5) (width 0.3) (layer F.Cu) (net 9))
   (segment (start 189.3 80.5) (end 189.3 81.45) (width 0.3) (layer F.Cu) (net 9))
+  (segment (start 140.5 92.350001) (end 140.5 89.5) (width 0.5) (layer B.Cu) (net 9))
+  (segment (start 141.149999 93) (end 140.5 92.350001) (width 0.5) (layer B.Cu) (net 9))
+  (segment (start 155.25 92) (end 154.25 93) (width 0.5) (layer B.Cu) (net 9))
+  (segment (start 154.25 93) (end 141.149999 93) (width 0.5) (layer B.Cu) (net 9))
   (segment (start 139.87 67.78) (end 139.87 65.98) (width 0.3) (layer F.Cu) (net 10))
   (segment (start 145.66 68.41) (end 140.5 68.41) (width 0.3) (layer F.Cu) (net 10))
