File: hardware/pcb/audiostick.sch (EAGLE design)
At the start: 61 parts, among them IC1 TPS73633MBDV, IC3 PCM5102ASW, IC5 AP22804W5, IC6 TINY13V-10SSU, J1 AVRISP6TH127, J2 AUDIO_JACK_3.5MM_PTH, J3 USB-B, SW1 EVQP7, T1 BC850

Commit message: Finish schematic/layout changes
Parts:
- removed J1: AVRISP6TH127, AWJLEagleLib:AVRISP6TH127
- added J4: AVRISP, AudioStick:AVRISP
- C14, C3: value 4u7 -> 2u2
- IC1: value TPS73633MBDV -> AP2127K; device AudioStick:TPS73633MBDV -> AudioStick:AP2127K
- R10: value 100K -> 10K
Connections:
- net !RST: now also J4.!RST; no longer J1.RST
- net +3V3: now also J4.VTG; no longer J1.VTG
- net +5V: now also IC1.!EN; no longer IC1.EN
- net ACK: now also J4.MISO; no longer J1.MISO
- net GND: now also J4.GND; no longer J1.GND
- net LED: now also J4.MOSI; no longer J1.MOSI
- net N$16: now also IC1.NC; no longer IC1.NR
- net SW: now also J4.SCK; no longer J1.SCK
Other:
- moved on the sheet: C16, IC1
